Commit message: update g1 23dof

File: unitree_g1/urdf/g1_23dof.urdf (robot description, URDF)
Before this commit: robot g1_23dof, 33 links, 32 joints
Links:
- removed link d435_link
- removed link imu_in_pelvis
- removed link imu_in_torso
- removed link mid360_link
- added link imu_link
Joints:
- removed joint d435_joint
- removed joint imu_in_pelvis_joint
- removed joint imu_in_torso_joint
- removed joint mid360_joint
- added joint imu_joint: type fixed, parent torso_link, child imu_link, origin xyz=-0.03959 -0.00224 0.13792 rpy=0 0 0
- joint left_wrist_roll_joint: type revolute -> fixed
- joint right_wrist_roll_joint: type revolute -> fixed
